File: code/nader/PCB/Bikota.brd (EAGLE design)
At the start: 160 x 100 mm, 6 parts

Commit message: Updated schematic and board files.
Parts:
- added C1: (no value), rcl:C0805
- added FUSE: MF-SMDF050, fuse:MF-SMDF050
- added JP1: Power, pinhead:1X02
- added JP2, JP3: (no value), pinhead:1X20
- added JP4, JP5, JP6, JP7: (no value), pinhead:1X01
- added LED1: (no value), led:CHIPLED_0805
- added Q1: IRLML6244, bytewerk:SOT23
- added R1: 100, rcl:R0805
- added R2, R7: 500, rcl:R0805
- added R3, R5, R6: 100K, rcl:R0805
- added R4: 1K, rcl:R0805
- added SG1: F/CM12P, buzzer:F/CM12P
- added U$7: EPAPERDISPLAY2.9, Bikota:EPAPERDISPLAY2.9
- added U$8: U1V11F5, Bikota:U1V11F5
- moved U$5 71.1 mm to (61.0, 81.3), turned to 90 degrees
- moved U$4 56.2 mm to (44.5, 20.3), turned to 0 degrees
- moved U$6 53.4 mm to (29.2, 25.4)
- moved U$2 46.0 mm to (62.2, 17.8), turned to 180 degrees
- moved U$1 38.6 mm to (41.9, 54.6)
- moved U$3 36.1 mm to (62.2, 91.4)
Connections:
- removed net ESP32_5V: U$1.ESP32_5V, U$2.P$1
- removed net ESP_3V3: U$1.ESP32_3V3
- new net BUZZER: JP3.15, SG1.-, U$1.GPIO2
- new net ESP3V3: JP2.20, R1.1, U$1.ESP32_3V3, U$4.P$1
- new net ESP5V: JP2.2, LED1.A, U$1.ESP32_5V, U$2.P$1, U$3.P$1, U$5.P$1, U$6.P$1, U$8.P$1
- new net MOSFET: JP2.8, R2.1, U$1.GPIO12
- new net MOSFET_GND: Q1.3, R4.1, U$3.P$4, U$4.P$2, U$5.P$2, U$6.P$2
- new net N$11: JP2.6, U$1.GPIO13
- new net N$14: JP2.3, U$1.CMD
- new net N$15: JP2.1, U$1.SPK+
- new net N$16: JP4.1, U$1.SPK-
- new net N$17: JP6.1, R7.2
- new net N$18: JP3.2, U$1.GPIO23
- new net N$2: R1.2, SG1.+
- new net N$20: JP3.4, U$1.TXD
- new net N$21: JP3.5, U$1.RXD
- new net N$23: JP3.10, U$1.GPIO5
- new net N$24: JP3.11, U$1.NC3
- new net N$25: JP3.12, U$1.NC2
- new net N$26: JP3.13, U$1.GPIO4
- new net N$27: JP3.14, U$1.GPIO0
- new net N$28: JP3.16, U$1.GPIO15
- new net N$29: JP3.17, U$1.SD1
- new net N$3: JP2.19, U$1.P$2
- new net N$30: JP3.18, U$1.SD0
- new net N$31: JP3.19, U$1.CLK
- new net N$32: JP3.20, U$1.MIC-
- new net N$33: JP5.1, U$1.MIC+
- new net N$412: U$7.P$1
- new net N$413: U$7.P$2
- new net N$414: U$7.P$3
- new net N$415: U$7.P$4
- new net N$416: U$7.P$5
- new net N$417: U$7.P$6
- new net N$418: U$7.P$7
- new net N$419: U$7.P$8
- new net N$5: JP2.14, U$1.GPIO32
- new net N$6: LED1.C, R4.2
- new net SVN: C1.1, JP2.17, R5.1, R6.2, U$1.SVN
- new net VBAT+: JP1.1, R5.2, U$8.P$3
- net ACC_INT: now also JP2.9
- net GND: now also C1.2, JP1.2, JP2.7, JP3.1, JP3.7, Q1.2, R3.2, R6.1, R7.1, U$8.P$2
- net GPS_TX: now also JP2.15
- net N$1: now also JP2.16, U$1.GPIO34; no longer U$3.P$1
- net N$10: now also JP2.10, U$1.GPIO27; no longer U$4.P$1
- net N$12: now also JP2.5, U$1.SD2; no longer U$5.P$2
- net N$13: now also JP2.4, U$1.SD3; no longer U$5.P$1
- net N$4: now also Q1.1, R2.2, R3.1; no longer U$3.P$4
- net N$7: now also JP2.13, U$1.GPIO33; no longer U$6.P$2
- net N$8: now also JP2.12, U$1.GPIO25; no longer U$6.P$1
- net N$9: now also JP2.11, U$1.GPIO26; no longer U$4.P$2
- net PM10: now also JP3.9
- net PM25: now also JP3.8
- net SCL: now also JP3.3
- net SDA: now also JP3.6
- net SVP: now also JP2.18
Routing:
- net GND: track 113.6 -> 0.00 mm, vias 1 -> 0
- net SCL: track 104.5 -> 0.00 mm
- net SDA: track 95.9 -> 0.00 mm
- net ACC_INT: track 74.2 -> 0.00 mm, vias 1 -> 0
- net ESP32_5V: track 48.0 -> 0.00 mm
- net SVP: track 25.1 -> 0.00 mm
- net PM10: track 10.5 -> 0.00 mm
- net PM25: track 10.5 -> 0.00 mm
- net GPS_TX: track 9.20 -> 0.00 mm
Other:
- board size 160 x 100 mm -> 109.2 x 100 mm

Commit message: Update PCB and SCH
Parts:
- removed FUSE: MF-SMDF050, fuse:MF-SMDF050
- added F1: 1206L, ptc-littlefuse:1206L
- moved U$7 79.6 mm to (54.6, 66.8), turned to 90 degrees
- moved R5 22.9 mm to (41.9, 71.1), turned to 90 degrees
- moved U$3 21.7 mm to (69.8, 71.1)
- moved JP1 18.2 mm to (11.4, 69.8)
- moved U$8 17.6 mm to (21.6, 70.2)
- moved R6 16.7 mm to (45.7, 71.1), turned to 270 degrees
- moved R7 15.5 mm to (38.1, 71.1)
- moved LED1 14.6 mm to (9.91, 60.8), turned to 270 degrees
- moved JP6 14.2 mm to (38.1, 66.0)
- moved R4 13.1 mm to (15.2, 61.0), turned to 180 degrees
- moved JP2 12.3 mm to (49.5, 61.6)
- moved JP4 12.3 mm to (22.9, 61.6)
- moved C1 12.0 mm to (49.5, 71.1), turned to 90 degrees
- moved JP7 10.5 mm to (40.6, 19.1), turned to 180 degrees
- moved U$1 10.5 mm to (44.5, 44.5)
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Connections:
- removed net N$1: JP2.16, U$1.GPIO34
- removed net N$28: JP3.16, U$1.GPIO15
- removed net N$412: U$7.P$1
- removed net N$413: U$7.P$2
- removed net N$414: U$7.P$3
- removed net N$415: U$7.P$4
- removed net N$416: U$7.P$5
- removed net N$417: U$7.P$6
- removed net N$419: U$7.P$8
- removed net N$5: JP2.14, U$1.GPIO32
- removed net N$7: JP2.13, U$1.GPIO33
- removed net N$8: JP2.12, U$1.GPIO25
- new net EP_BUSY: JP2.16, U$1.GPIO34, U$7.P$8
- new net EP_CLK: JP2.12, U$1.GPIO25, U$7.P$4
- new net EP_CS: JP2.13, U$1.GPIO33, U$7.P$5
- new net EP_DC: JP2.14, U$1.GPIO32, U$7.P$6
- new net EP_DIN: JP3.16, U$1.GPIO15, U$7.P$3
- new net N$41: F1.P$2, JP1.1
- net ESP3V3: now also U$7.P$1
- net GND: now also JP7.1, U$7.P$2
- net VBAT+: now also F1.P$1; no longer JP1.1
Routing:
- net ESP5V: track 0.00 -> 159.9 mm, vias 0 -> 2
- net MOSFET_GND: track 0.00 -> 129.5 mm, vias 0 -> 2
- net ESP3V3: track 0.00 -> 93.8 mm
- net GND: track 0.00 -> 62.6 mm
- net EP_DIN: track 0.00 -> 50.6 mm, vias 0 -> 2
- net ACC_INT: track 0.00 -> 47.7 mm, vias 0 -> 2
- net SVN: track 0.00 -> 34.7 mm, vias 0 -> 1
- net SCL: track 0.00 -> 34.2 mm
- net BUZZER: track 0.00 -> 32.4 mm
- net SDA: track 0.00 -> 28.6 mm
- net PM25: track 0.00 -> 28.5 mm
- net PM10: track 0.00 -> 28.5 mm
- net VBAT+: track 0.00 -> 26.9 mm
- net GPS_TX: track 0.00 -> 21.1 mm, vias 0 -> 1
- net MOSFET: track 0.00 -> 19.8 mm
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- added copper zone on layer 1, net GND
- added copper zone on layer 16, net GND
Other:
- board size 109.2 x 100 mm -> 83.8 x 78.4 mm
